File: Alice/Alice.sch (EAGLE design)
At the start: 17 parts, among them Q1 J305, Q2 2N5087, Q3 2N5087, X1 Mic, X2 XLR

Commit message: Done!
Parts:
- C1: value 10uF -> .47uF; device adafruit:CPOL-USE1.8-4 -> adafruit:C-US075-052X106
- C2: value 68uF -> .47uF; device adafruit:CPOL-USE3.5-10 -> adafruit:C-US075-052X106
- C3: value .47uF -> 68uF; device adafruit:C-US075-052X106 -> adafruit:CPOL-USE3.5-10
- C4: value .47uF -> 10uF; device adafruit:C-US075-052X106 -> adafruit:CPOL-USE1.8-4
- renumbered R8 to R7
Connections:
- net N$1: now also C1.1; no longer C3.1
- net N$3: now also C3.+; no longer C2.+
- net N$4: now also C2.1; no longer C4.1
- net N$6: now also C1.2; no longer C3.2
- net N$7: now also C2.2; no longer C4.2
- net N$9: now also C4.+; no longer C1.+
- net XLR-1: now also C3.-, C4.-; no longer C1.-, C2.-
